File: Hardware/Kicad/CAT FLAP/CatFlap_PCB/CatFlap_PCB.kicad_pcb (KiCad board)
At the start: 2 copper layers, 196 x 25 mm, 77 parts, among them J1 Conn_01x08, J2 Conn_01x03, J3 Battery pack, J4 Conn_01x03_Socket, J5 Conn_01x03, J6 Conn_01x02, J8 Conn_01x20, J9 Conn_01x20, M1 Motor_DC, Q1 NX3008CBKS, Q2 Q_PMOS_DGS, SW1 SW_Push, SW2 SW_Push, SW3 SW_Push, T1 NX3008NBKS, T2 NX3008NBKS, T3 NX3008NBKS, U1 LM358_DFN, U2 DRV8837DSGR, U3 TPS62132

Commit message: Fixed things from first rev of PCB
Parts:
- removed JP4: SolderJumper_3_Bridged12, Jumper:SolderJumper-3_P1.3mm_Bridged12_RoundedPad1.0x1.5mm
- removed Q2: Q_PMOS_DGS, Package_TO_SOT_SMD:SOT-23
- added Q3: Q_PMOS_GSD, Package_TO_SOT_SMD:SOT-23, F.Cu at (109.5, 74.4)
- added R27: 330k, Resistor_SMD:R_0603_1608Metric, F.Cu at (93.0, 74.7)
- added R28: 330k, Resistor_SMD:R_0603_1608Metric, F.Cu at (110.1, 82.5)
- added R29: 330k, Resistor_SMD:R_0603_1608Metric, F.Cu at (90.7, 81.5)
- Q1: footprint Package_TO_SOT_SMD:TSOT-23-6 -> Package_TO_SOT_SMD:SOT-363_SC-70-6
Connections:
- J8 pad 11: Reset -> /RUN
- U2 pad 7: Net-(JP4-C) -> M_SLEEP
Routing:
- net Reset: track 65.9 -> 63.1 mm
- net Net-(JP4-C): track 2.67 -> 0.00 mm
- net LED_B: track 53.5 -> 55.2 mm
- net M_SLEEP: track 31.0 -> 32.5 mm
- net Net-(J3-V+): track 177.5 -> 176.0 mm
- net LED_G: track 58.2 -> 59.7 mm
- net LED_R: track 66.0 -> 67.5 mm
- net VDD: track 177.8 -> 178.6 mm
- net GND: track 71.7 -> 72.1 mm, vias 162 -> 161
